File: asic.kicad_sch (KiCad schematic)
At the start: 122 parts, among them U10 MCP1824T-1202E/OT, U11 MCP1824T-1202E/OT, U12 MCP1824T-0802E, U13 MCP1824T-0802E, U7 SN74AXC4T774, U8 25MHz, U9 25MHz

Commit message: power sheet schematic cleanup
Parts:
- C106, C115, C129, C135, C141, C45: value 100nf -> 0.1uF
