File: power.kicad_sch (KiCad schematic)
At the start: 134 parts, among them U18 TPS62933, U19 TPS62933, U3 TPS546D24S, U4 TPS546D24S, U5 TPS546D24S, U6 TPS546D24S

Commit message: fix KiCad trailing space warning
Parts:
- C103, C105, C151, C152, C164, C165, C167, C168, C69, C70, C73, C74, C75, C76, C80, C82: Manufacturer muRata -> (none)

Commit message: power sheet schematic cleanup
Parts:
- C19, C22, C25, C42: value 100nf -> 0.1uF
Other:
- moved on the sheet: C10, C101, C103, C104, C105, C107, C11, C12, C13, C139, C14, C140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
